File: hall-matrix-key/hall-matrix-key.kicad_pcb (KiCad board)
At the start: 2 copper layers, 176.5 x 59.9 mm, 18 parts, among them J1 Conn_01x06_Pin, J2 Conn_01x06_Pin, J3 Conn_01x06_Pin, J4 Conn_01x06_Pin, J5 Conn_01x01_Pin, J6 Conn_01x08_Pin

Commit message: second batch with corrections (purple)
Parts:
- J1: footprint robodisk:hall-matrix-selector-switch_base -> Library:hall-matrix-selector-switch_base
- J3: footprint robodisk:hall-matrix-selector-switch_knob -> Library:hall-matrix-selector-switch_rotator
- moved D3 39.9 mm to (73.9, 117.0), turned to -130 degrees
- moved D4 39.6 mm to (81.4, 69.1), turned to 110 degrees
- moved R3 36.6 mm to (75.4, 115.2), turned to 140 degrees
- moved R4 36.3 mm to (82.2, 71.2), turned to 20 degrees
- moved D6 14.6 mm to (81.4, 121.4), turned to -110 degrees
- moved D5 14.6 mm to (77.4, 119.4), turned to -120 degrees
- moved D2 14.4 mm to (77.5, 70.9), turned to 120 degrees
- moved D1 14.3 mm to (73.9, 73.5), turned to 130 degrees
- moved R6 13.4 mm to (82.2, 119.1), turned to 160 degrees
- moved R5 13.3 mm to (78.7, 117.4), turned to 150 degrees
- moved R2 13.2 mm to (78.6, 72.9), turned to 30 degrees
- moved R1 13.2 mm to (75.4, 75.3), turned to 40 degrees
- turned J1 to 150 degrees
- turned J3 to 150 degrees
Connections:
- D1 pad 2: /I1 -> /I3
- D3 pad 2: /I3 -> /O1
- D4 pad 2: /O1 -> /I1
- J1 pad 1: /O1 -> /I1
- J1 pad 2: /I1 -> /I2
- J1 pad 3: /I2 -> /I3
- J1 pad 4: /O2 -> /O1
- J1 pad 5: /O3 -> /O2
- J1 pad 6: /I3 -> /O3
- J3 pad 4: Net-(J3-Pin_3) -> Net-(J3-Pin_1)
- J3 pad 6: Net-(J3-Pin_1) -> Net-(J3-Pin_3)
- J4 pad 1: /O1 -> /I1
- J4 pad 2: /I1 -> /O1
- J4 pad 3: /O2 -> /I2
- J4 pad 4: /I2 -> /O2
- J4 pad 5: /O3 -> /I3
- J4 pad 6: /I3 -> /O3
Routing:
- net GND: track 21.6 -> 0.13 mm, vias 13 -> 7
- net /O2: track 116.3 -> 98.5 mm
- net /O1: track 113.2 -> 126.5 mm
- net /O3: track 113.2 -> 105.5 mm
- net /I2: track 108.4 -> 104.2 mm
- net /I3: track 105.1 -> 107.3 mm
- net /I1: track 112.7 -> 112.1 mm
Other:
- board size 176.5 x 59.9 mm -> 178 x 59.9 mm
- board text added: "IN"
- board text added: "OUT"
- board text removed: "IN (red)"
- board text removed: "OUT (green)"
