File: hall-matrix-key/hall-matrix-key.kicad_sch (KiCad schematic)
At the start: 6 parts, among them J1 Conn_01x06_Pin, J2 Conn_01x06_Pin, J3 Conn_01x06_Pin, J4 Conn_01x06_Pin, J5 Conn_01x01_Pin, J6 Conn_01x08_Pin

Commit message: stale changes
Parts:
- added D1, D2, D3, D4, D5, D6: LED, LED_SMD:LED_LiteOn_LTST-S326, symbol Device:LED
- added R1, R2, R3, R4, R5, R6: R, Resistor_SMD:R_0805_2012Metric_Pad1.20x1.40mm_HandSolder, symbol Device:R
- J5: footprint (none) -> robodisk:keyhole
Connections:
- net GND: now also R1.2, R2.2, R3.2, R4.2, R5.2, R6.2
- net I1: now also D1.2 (A)
- net I2: now also D2.2 (A)
- net I3: now also D3.2 (A)
- net O1: now also D4.2 (A)
- net O2: now also D5.2 (A)
- net O3: now also D6.2 (A)
- new net: D1.1 (K), R1.1
- new net: D3.1 (K), R3.1
- new net: D4.1 (K), R4.1
- new net: D2.1 (K), R2.1
- new net: D5.1 (K), R5.1
- new net: D6.1 (K), R6.1
Other:
- note added: "6x Pogo pins ie. Mill-Max 823-22-06-10-000-101 Digikey: ED8180-ND"
- note added: "Center axis: Würth Elektronic 7466003R Digikey: 732-5647-2-ND"
- note added: "Required: 6x Pogo pins for contact Optional: 1-4x Pogo pins for stab & position locking MFGR Ref: Mill-Max 0980-0-15-20-75-14-11-0 Digikey: ED5073-N"
- moved on the sheet: J1, J3, J5

Commit message: second batch with corrections (purple)
Connections:
- net I1: now also D4.2 (A), J1.1 (Pin_1), J4.1 (Pin_1); no longer D1.2 (A), J1.2 (Pin_2), J4.2 (Pin_2)
- net I2: now also J1.2 (Pin_2), J4.3 (Pin_3); no longer J1.3 (Pin_3), J4.4 (Pin_4)
- net I3: now also D1.2 (A), J1.3 (Pin_3), J4.5 (Pin_5); no longer D3.2 (A), J1.6 (Pin_6), J4.6 (Pin_6)
- net O1: now also D3.2 (A), J1.4 (Pin_4), J4.2 (Pin_2); no longer D4.2 (A), J1.1 (Pin_1), J4.1 (Pin_1)
- net O2: now also J1.5 (Pin_5), J4.4 (Pin_4); no longer J1.4 (Pin_4), J4.3 (Pin_3)
- net O3: now also J1.6 (Pin_6), J4.6 (Pin_6); no longer J1.5 (Pin_5), J4.5 (Pin_5)
- net at J3.1 (Pin_1): now also J3.4 (Pin_4); no longer J3.6 (Pin_6)
- net at J3.3 (Pin_3): now also J3.6 (Pin_6); no longer J3.4 (Pin_4)
Other:
- moved on the sheet: D1, D2, D3, D5, D6, J2, R1, R2, R3, R5, R6
